File: sensorboard_due/sensorboard_due.sch (KiCad schematic (older format))
At the start: 35 parts

Commit message: working electrical rules - but a bit hacky
Parts:
- gave numbers to parts that had none: 35
Connections:
- wire segments 98 -> 116
- no-connect marks 85 -> 108
Other:
- moved on the sheet: D1, D2, D3, D4, D5, D6, J1, J6, R1, R2, R3, R4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
