File: sensorboard_due_v2/sensorboard_due.sch (KiCad schematic (older format))
At the start: 30 parts, among them J1 LED_PANEL, J11 DHT22_Conn, J12 DHT22_Conn, J13 DHT22_Conn, J14 DHT22_Conn, J15 DHT22_Conn, J16 DHT22_Conn, J17 DHT22_Conn, J18 DHT22_Conn, J2 I2C_SLAVE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

Commit message: halfway through ... need to route pcb
Parts:
- removed H3: MPU-9250_Breakout, arduino_sensors:MPU-9250_Breakout, symbol arduino_sensors:MPU-9250_Breakout
- removed J17, J18: DHT22_Conn, Connector_Molex_70553:70553-0002_3P, symbol arduino_sensors:DHT22_Conn
- removed J24: MPU-9250_Conn, Connector_Molex_70553:70553-0004_5P, symbol arduino_sensors:MPU-9250_Conn
- removed R7, R8: 10k, symbol Device:R
- added J5: GPS_UBLOX_NEO6M, Connector_Molex_70553:70553-0038_4P, symbol arduino_sensors:GPS_UBLOX_NEO6M
- J1: footprint (none) -> Connector_Molex_70553:70553-0042_8P
- R1, R2, R3, R4, R5, R6: footprint (none) -> Resistor_THT:R_Axial_DIN0207_L6.3mm_D2.5mm_P7.62mm_Horizontal
- renumbered J22 to J21, J23 to J22, J25 to J23, J26 to J24
Connections:
- net +3V3: now also J5.1 (Vcc)
- net A0_OUT: now also J1.8 (Pin_8); no longer J1.1 (Pin_1)
- net A1_OUT: now also J1.7 (Pin_7); no longer J1.2 (Pin_2)
- net A2_OUT: now also J1.6 (Pin_6); no longer J1.3 (Pin_3)
- net A3_OUT: now also J1.5 (Pin_5); no longer J1.4 (Pin_4)
- net A4_OUT: now also J1.4 (Pin_4); no longer J1.5 (Pin_5)
- net A5_OUT: now also J1.3 (Pin_3); no longer J1.6 (Pin_6)
- net A6_OUT: now also J1.2 (Pin_2); no longer J1.7 (Pin_7)
- net GND: now also J1.1 (Pin_1), J5.4 (GND); no longer J1.8 (Pin_8)
- net MPU_1: now also J21.5 (AD0/SD0)
- net MPU_2: now also J22.5 (AD0/SD0); no longer J21.5 (AD0/SD0)
- net MPU_3: now also J23.5 (AD0/SD0); no longer J22.5 (AD0/SD0)
- net MPU_4: now also J24.5 (AD0/SD0)
- net at PCB1.16 (16(TX2)): now also J5.2 (RX)
- net at PCB1.17 (17(RX2)): now also J5.3 (TX)
- net DHT_7: no longer names the net of PCB1.35
- net DHT_8: no longer names the net of PCB1.37
- net MPU_5: no longer names the net of PCB1.30
- net MPU_5: no longer J23.5 (AD0/SD0)
- net MPU_6: no longer names the net of PCB1.32
- net MPU_6: no longer J24.5 (AD0/SD0)
- no-connect marks 67 -> 63
Other:
- note removed: "Pin no. scheme:\nright to left,\nanticlockwise"
- moved on the sheet: J1, J4, U1
