File: sensorboard_due_v2/sensorboard_due.sch (KiCad schematic (older format))
At the start: 30 parts, among them J1 LED_PANEL, J11 DHT22, J12 DHT22, J13 DHT22, J14 DHT22, J15 DHT22, J16 DHT22, J17 DHT22, J18 DHT22, J2 I2C_SLAVE, J22 MPU-9250_Breakout, J23 MPU-9250_Breakout, J24 MPU-9250_Breakout, J25 MPU-9250_Breakout, J26 MPU-9250_Breakout, J3 WATCHDOG, J4 GPS_UBLOX_NEO6M, U1 HSCDANN001BA2A3

Commit message: modified molex connectors to be datasheet compliant
Parts:
- removed J11, J12, J13, J14, J15, J16, J17, J18: DHT22, symbol arduino_sensors:DHT22
- removed J22, J23, J24, J25, J26: MPU-9250_Breakout, symbol arduino_sensors:MPU-9250_Breakout
- added J11, J12, J13, J14, J15, J16, J17, J18: DHT22_Conn, Connector_Molex_70553:70553-0002_3P, symbol arduino_sensors:DHT22_Conn
- added J22, J23, J24, J25, J26: MPU-9250_Conn, Connector_Molex_70553:70553-0004_5P, symbol arduino_sensors:MPU-9250_Conn
- J1: symbol Connector_Generic:Conn_01x07 -> Connector_Generic:Conn_01x08
- J2: footprint (none) -> Connector_Molex_70553:70553-0002_3P
- J3: footprint (none) -> Connector_Molex_70553:70553-0001_2P
- J4: footprint (none) -> Connector_Molex_70553:70553-0038_4P
- renumbered R7 to R1, R8 to R2, R9 to R3, R10 to R4, R3 to R5, R4 to R6, R1 to R7, R2 to R8
Connections:
- net labels added: A6_OUT
- wire segments 126 -> 147
- no-connect marks 98 -> 67
Other:
- note added: "Use dynamic addr selection \nto prevent I2C conflicts \nwith RTC, other MPUs."
- note removed: "Use dynamic addr selection to prevent\nI2C conflicts with RTC, other MPUs."
- moved on the sheet: R1, R2, R3, R4, R5, R6

Commit message: Sync
Parts:
- removed J11, J12, J13, J14, J15, J16, J17, J18: DHT22_Conn, Connector_Molex_70553:70553-0002_3P, symbol arduino_sensors:DHT22_Conn
- removed R1, R2, R3, R4, R5, R6, R7, R8: 10k, symbol Device:R
Connections:
- net DHT_1 renamed RTD_1_CS
- net DHT_2 renamed RTD_2_CS
- net DHT_3: no longer names the net of PCB1.27
- net DHT_4: no longer names the net of PCB1.29
- net DHT_5: no longer names the net of PCB1.31
- net DHT_6: no longer names the net of PCB1.33
- net DHT_7: no longer names the net of PCB1.35
- net DHT_8: no longer names the net of PCB1.37
Other:
- note removed: "Temperature/Humidity;\nnot necessarily on-board"

Commit message: asdasd
Parts:
- removed H1: SD_Card_Breakout, arduino_sensors:SD_Card_Breakout, symbol arduino_sensors:SD_Card_Breakout
- removed H3: MPU-9250_Breakout, arduino_sensors:MPU-9250_Breakout, symbol arduino_sensors:MPU-9250_Breakout
- removed J1: LED_PANEL, symbol Connector_Generic:Conn_01x08
- removed J22, J23, J24, J25, J26: MPU-9250_Conn, Connector_Molex_70553:70553-0004_5P, symbol arduino_sensors:MPU-9250_Conn
- removed J3: WATCHDOG, Connector_Molex_70553:70553-0001_2P, symbol Connector_Generic:Conn_01x02
- added C5, C6: 0.1u, Capacitor_SMD:C_0402_1005Metric, symbol Device:C
- added H1: MPU-9250_Breakout, arduino_sensors:MPU-9250_Breakout, symbol arduino_sensors:MPU-9250_Breakout
- added J5: Micro_SD_Card, Connector_Card:microSD_HC_Hirose_DM3BT-DSF-PEJS, symbol Connector:Micro_SD_Card
Connections:
- net labels added: MISO, MOSI, SCK
- net labels removed: A0_OUT, A1_OUT, A2_OUT, A3_OUT, A4_OUT, A5_OUT, A6_OUT
- wire segments 85 -> 69
- no-connect marks 67 -> 63
Other:
- note removed: "MPU: \nI2C 0x68/0x69"
- note removed: "On-board SPI slave devices"
- note removed: "Pin no. scheme:\nright to left,\nanticlockwise"
- note removed: "Use dynamic addr selection \nto prevent I2C conflicts \nwith RTC, other MPUs."
