File: sensorboard_due_v2/file60B83ABE.sch (KiCad schematic (older format))
At the start: 10 parts, among them J3 Conn_01x03_Male, J6 Conn_01x03_Male, U2 MAX31865AAP+, U3 MAX31865AAP+

Commit message: PCB layout
Parts:
- C1, C2, C3, C4: footprint Capacitor_SMD:C_0402_1005Metric -> Capacitor_SMD:C_0805_2012Metric_Pad1.15x1.40mm_HandSolder
Changed lines of the file:
@@
 F 0 "C1" H 2015 2796 50  0000 L CNN
 F 1 "0.1u" H 2015 2705 50  0000 L CNN
-F 2 "Capacitor_SMD:C_0402_1005Metric" H 1938 2600 50  0001 C CNN
+F 2 "Capacitor_SMD:C_0805_2012Metric_Pad1.15x1.40mm_HandSolder" H 1938 2600 50  0001 C CNN
 F 3 "~" H 1900 2750 50  0001 C CNN
 	1    1900 2750
@@
 F 0 "C2" H 3285 2796 50  0000 R CNN
 F 1 "0.1u" H 3285 2705 50  0000 R CNN
-F 2 "Capacitor_SMD:C_0402_1005Metric" H 3438 2600 50  0001 C CNN
+F 2 "Capacitor_SMD:C_0805_2012Metric_Pad1.15x1.40mm_HandSolder" H 3438 2600 50  0001 C CNN
 F 3 "~" H 3400 2750 50  0001 C CNN
 	1    3400 2750
@@
 F 0 "C3" H 5515 2796 50  0000 L CNN
 F 1 "0.1u" H 5515 2705 50  0000 L CNN
-F 2 "Capacitor_SMD:C_0402_1005Metric" H 5438 2600 50  0001 C CNN
+F 2 "Capacitor_SMD:C_0805_2012Metric_Pad1.15x1.40mm_HandSolder" H 5438 2600 50  0001 C CNN
 F 3 "~" H 5400 2750 50  0001 C CNN
 	1    5400 2750
@@
 F 0 "C4" H 6785 2796 50  0000 R CNN
 F 1 "0.1u" H 6785 2705 50  0000 R CNN
-F 2 "Capacitor_SMD:C_0402_1005Metric" H 6938 2600 50  0001 C CNN
+F 2 "Capacitor_SMD:C_0805_2012Metric_Pad1.15x1.40mm_HandSolder" H 6938 2600 50  0001 C CNN
 F 3 "~" H 6900 2750 50  0001 C CNN
 	1    6900 2750

Commit message: stuff
Parts:
- added C7, C8: 0.1u, Capacitor_SMD:C_0805_2012Metric_Pad1.15x1.40mm_HandSolder, symbol Device:C
Connections:
- wire segments 66 -> 58
- no-connect marks 0 -> 2
Other:
- moved on the sheet: J3
Changed lines of the file:
@@
 	3100 3100 3150 3100
 Wire Wire Line
-	3750 3350 3750 3400
-Wire Wire Line
 	3750 3400 3650 3400
-Connection ~ 3750 3400
 Wire Wire Line
 	3100 3200 3150 3200
@@
 	3650 3400 3100 3400
 Wire Wire Line
-	3550 3550 3550 3500
-Wire Wire Line
-	3550 3500 3250 3500
-Wire Wire Line
-	3550 3900 3100 3900
-Wire Wire Line
-	3100 3700 3450 3700
-Wire Wire Line
-	3450 3700 3450 3650
-Wire Wire Line
-	3550 3750 3350 3750
-Wire Wire Line
-	3350 3750 3350 3800
+	3550 3900 3350 3900
 Wire Wire Line
 	3350 3800 3100 3800
@@
 	6600 3100 6650 3100
 Wire Wire Line
-	7250 3350 7250 3400
-Wire Wire Line
 	7250 3400 7150 3400
-Connection ~ 7250 3400
 Wire Wire Line
 	6600 3200 6650 3200
@@
 	7150 3400 6600 3400
 Wire Wire Line
-	7050 3550 7050 3500
-Wire Wire Line
-	7050 3900 6600 3900
-Wire Wire Line
-	6600 3700 6950 3700
-Wire Wire Line
-	6950 3700 6950 3650
-Wire Wire Line
-	7050 3750 6850 3750
-Wire Wire Line
-	6850 3750 6850 3800
-Wire Wire Line
-	6850 3800 6600 3800
-Wire Wire Line
-	6750 3600 6600 3600
-Wire Wire Line
-	3550 3750 3550 3900
-Wire Wire Line
 	3250 3600 3250 3500
-Connection ~ 3250 3500
 Wire Wire Line
 	3250 3500 3100 3500
-Connection ~ 3550 3750
 $Comp
 L Connector:Conn_01x03_Male J3
 U 1 1 60A805EA
-P 4000 3650
-F 0 "J3" H 3972 3674 50  0000 R CNN
-F 1 "Conn_01x03_Male" H 3972 3583 50  0000 R CNN
-F 2 "Connector_Molex_70553:70553-0002_3P" H 4000 3650 50  0001 C CNN
-F 3 "~" H 4000 3650 50  0001 C CNN
-	1    4000 3650
-	-1   0    0    -1
-$EndComp
+P 4300 3600
+F 0 "J3" H 4272 3624 50  0000 R CNN
+F 1 "Conn_01x03_Male" H 4272 3533 50  0000 R CNN
+F 2 "Connector_Molex_70553:70553-0002_3P" H 4300 3600 50  0001 C CNN
+F 3 "~" H 4300 3600 50  0001 C CNN
+	1    4300 3600
+	-1   0    0    1
+$EndComp
+NoConn ~ 2200 3100
+NoConn ~ 5700 3100
+Connection ~ 3250 3500
+$Comp
+L Device:C C7
+U 1 1 60D14DB5
+P 3550 3700
+F 0 "C7" H 3665 3746 50  0000 L CNN
+F 1 "0.1u" H 3665 3655 50  0000 L CNN
+F 2 "Capacitor_SMD:C_0805_2012Metric_Pad1.15x1.40mm_HandSolder" H 3588 3550 50  0001 C CNN
+F 3 "~" H 3550 3700 50  0001 C CNN
+	1    3550 3700
+	1    0    0    -1
+$EndComp
+Wire Wire Line
+	3350 3800 3350 3900
+Connection ~ 3350 3900
+Wire Wire Line
+	3350 3900 3100 3900
+Wire Wire Line
+	3550 3900 3550 3850
+Wire Wire Line
+	4100 3700 4100 3900
+Wire Wire Line
+	4100 3900 3550 3900
+Connection ~ 3550 3900
+Wire Wire Line
+	3100 3700 3400 3700
+Wire Wire Line
+	3400 3700 3400 3550
+Wire Wire Line
+	3400 3550 3550 3550
+Wire Wire Line
+	3550 3550 3900 3550
+Wire Wire Line
+	3900 3550 3900 3600
+Wire Wire Line
+	3900 3600 4100 3600
+Connection ~ 3550 3550
+Wire Wire Line
+	3250 3500 4100 3500
+Wire Wire Line
+	7050 3900 6850 3900
+Wire Wire Line
+	6850 3800 6600 3800
+Wire Wire Line
+	6750 3600 6600 3600
+Wire Wire Line
+	6750 3600 6750 3500
+Wire Wire Line
+	6750 3500 6600 3500
 $Comp
 L Connector:Conn_01x03_Male J6
-U 1 1 60A866ED
-P 7500 3650
-F 0 "J6" H 7472 3674 50  0000 R CNN
-F 1 "Conn_01x03_Male" H 7472 3583 50  0000 R CNN
-F 2 "Connector_Molex_70553:70553-0002_3P" H 7500 3650 50  0001 C CNN
-F 3 "~" H 7500 3650 50  0001 C CNN
-	1    7500 3650
-	-1   0    0    -1
-$EndComp
-Wire Wire Line
-	7050 3500 6750 3500
-Wire Wire Line
-	6750 3600 6750 3500
+U 1 1 60D34292
+P 7800 3600
+F 0 "J6" H 7772 3624 50  0000 R CNN
+F 1 "Conn_01x03_Male" H 7772 3533 50  0000 R CNN
+F 2 "Connector_Molex_70553:70553-0002_3P" H 7800 3600 50  0001 C CNN
+F 3 "~" H 7800 3600 50  0001 C CNN
+	1    7800 3600
+	-1   0    0    1
+$EndComp
 Connection ~ 6750 3500
-Wire Wire Line
-	6750 3500 6600 3500
-Wire Wire Line
-	3550 3750 3700 3750
-Wire Wire Line
-	3700 3750 3700 3550
-Wire Wire Line
-	3700 3550 3800 3550
-Wire Wire Line
-	3450 3650 3800 3650
-Wire Wire Line
-	3550 3550 3650 3550
-Wire Wire Line
-	3650 3550 3650 3700
-Wire Wire Line
-	3650 3700 3800 3700
-Wire Wire Line
-	3800 3700 3800 3750
-Wire Wire Line
-	7050 3750 7050 3850
-Wire Wire Line
-	7300 3550 7150 3550
-Wire Wire Line
-	7150 3550 7150 3850
-Wire Wire Line
-	7150 3850 7050 3850
-Connection ~ 7050 3850
-Wire Wire Line
-	7050 3850 7050 3900
-Wire Wire Line
-	7050 3500 7200 3500
-Wire Wire Line
-	7200 3500 7200 3750
-Wire Wire Line
-	7200 3750 7300 3750
-Connection ~ 7050 3500
-Wire Wire Line
-	6950 3650 7300 3650
+$Comp
+L Device:C C8
+U 1 1 60D34299
+P 7050 3700
+F 0 "C8" H 7165 3746 50  0000 L CNN
+F 1 "0.1u" H 7165 3655 50  0000 L CNN
+F 2 "Capacitor_SMD:C_0805_2012Metric_Pad1.15x1.40mm_HandSolder" H 7088 3550 50  0001 C CNN
+F 3 "~" H 7050 3700 50  0001 C CNN
+	1    7050 3700
+	1    0    0    -1
+$EndComp
+Wire Wire Line
+	6850 3800 6850 3900
+Connection ~ 6850 3900
+Wire Wire Line
+	6850 3900 6600 3900
+Wire Wire Line
+	7050 3900 7050 3850
+Wire Wire Line
+	7600 3700 7600 3900
+Wire Wire Line
+	7600 3900 7050 3900
+Connection ~ 7050 3900
+Wire Wire Line
+	6600 3700 6900 3700
+Wire Wire Line
+	6900 3700 6900 3550
+Wire Wire Line
+	6900 3550 7050 3550
+Wire Wire Line
+	7050 3550 7400 3550
+Wire Wire Line
+	7400 3550 7400 3600
+Wire Wire Line
+	7400 3600 7600 3600
+Connection ~ 7050 3550
+Wire Wire Line
+	6750 3500 7600 3500
 $EndSCHEMATC

Commit message: incomplete pcb layout
Parts:
- removed J3, J6: Conn_01x03_Male, Connector_Molex_70553:70553-0002_3P, symbol Connector:Conn_01x03_Male
- added C10, C11, C12, C13, C14, C15, C16, C17, C18, C19, C20, C9: 0.1u, Capacitor_SMD:C_0805_2012Metric_Pad1.15x1.40mm_HandSolder, symbol Device:C
- added J1, J3, J6, J7, J8, J9: Conn_01x04_Male, Connector_JST:JST_XH_B4B-XH-A_1x04_P2.50mm_Vertical, symbol Connector:Conn_01x04_Male
- added JP11, JP13, JP14, JP17, JP18, JP20: SolderJumper_2_Open, Jumper:SolderJumper-2_P1.3mm_Open_Pad1.0x1.5mm, symbol Jumper:SolderJumper_2_Open
- added JP12, JP15, JP16, JP19, JP21, JP22: SolderJumper_3_Open, Jumper:SolderJumper-3_P1.3mm_Open_Pad1.0x1.5mm, symbol Jumper:SolderJumper_3_Open
- added R3, R4, R5, R6: 400, Resistor_SMD:R_0603_1608Metric_Pad1.05x0.95mm_HandSolder, symbol Device:R
- added U5, U6, U7, U8: MAX31865AAP+, Package_SO:SSOP-20_5.3x7.2mm_P0.65mm, symbol arduino_sensors:MAX31865AAP+
Connections:
- net +3V3: now also C8.1, C12.1, C13.1, C14.1, C15.1, C16.1, C17.1, C9.1, U5.2 (DVDD), U5.3 (VDD), U6.2 (DVDD), U6.3 (VDD), U7.2 (DVDD), U7.3 (VDD), U8.2 (DVDD), U8.3 (VDD)
- net GND: now also C8.2, C12.2, C13.2, C14.2, C15.2, C16.2, C17.2, C9.2, JP12.3 (B), JP15.3 (B), JP16.3 (B), JP19.3 (B), JP21.3 (B), JP22.3 (B), U5.13 (GND2), U5.18 (DGND), U5.19 (GND1), U6.13 (GND2), U6.18 (DGND), U6.19 (GND1), U7.13 (GND2), U7.18 (DGND), U7.19 (GND1), U8.13 (GND2), U8.18 (DGND), U8.19 (GND1)
- net MISO: now also U5.17 (SDO), U6.17 (SDO), U7.17 (SDO), U8.17 (SDO)
- net MOSI: now also U5.14 (SDI), U6.14 (SDI), U7.14 (SDI), U8.14 (SDI)
- net RTD_1_CS: now also U7.16 (~CS); no longer U2.16 (~CS)
- net RTD_2_CS: now also U2.16 (~CS); no longer U3.16 (~CS)
- net SCK: now also U5.15 (SCLK), U6.15 (SCLK), U7.15 (SCLK), U8.15 (SCLK)
- net at C7.2, U2.11 (RTDIN-): now also J1.2 (Pin_2), JP11.1 (A); no longer U2.12 (FORCE-)
- net at C7.1, U2.10 (RTDIN+): now also J1.3 (Pin_3)
- net at U2.8 (FORCE+): now also J1.4 (Pin_4), JP12.1 (A); no longer U2.9 (FORCE2)
- net at U3.10 (RTDIN+): now also C10.1, J3.3 (Pin_3); no longer C8.1
- net at U3.8 (FORCE+): now also J3.4 (Pin_4), JP15.1 (A); no longer U3.9 (FORCE2)
- new net: J1.1 (Pin_1), JP11.2 (B), U2.12 (FORCE-)
- new net: JP12.2 (C), U2.9 (FORCE2)
- new net: C11.1, J6.3 (Pin_3), U5.10 (RTDIN+)
- new net: C11.2, J6.2 (Pin_2), JP14.1 (A), U5.11 (RTDIN-)
- new net: J6.1 (Pin_1), JP14.2 (B), U5.12 (FORCE-)
- new net: R3.1, U5.4 (BIAS), U5.5 (REFIN+)
- new net: R3.2, U5.6 (REFIN-), U5.7 (ISENSOR)
- new net: J6.4 (Pin_4), JP16.1 (A), U5.8 (FORCE+)
- new net: JP16.2 (C), U5.9 (FORCE2)
- new net: C10.2, J3.2 (Pin_2), JP13.1 (A), U3.11 (RTDIN-)
- new net: J3.1 (Pin_1), JP13.2 (B), U3.12 (FORCE-)
- new net: JP15.2 (C), U3.9 (FORCE2)
- new net: C20.1, J9.3 (Pin_3), U8.10 (RTDIN+)
- new net: C20.2, J9.2 (Pin_2), JP20.1 (A), U8.11 (RTDIN-)
- new net: J9.1 (Pin_1), JP20.2 (B), U8.12 (FORCE-)
- new net: R6.1, U8.4 (BIAS), U8.5 (REFIN+)
- new net: R6.2, U8.6 (REFIN-), U8.7 (ISENSOR)
- new net: J9.4 (Pin_4), JP22.1 (A), U8.8 (FORCE+)
- new net: JP22.2 (C), U8.9 (FORCE2)
- new net: C19.1, J8.3 (Pin_3), U7.10 (RTDIN+)
- new net: C19.2, J8.2 (Pin_2), JP18.1 (A), U7.11 (RTDIN-)
- new net: J8.1 (Pin_1), JP18.2 (B), U7.12 (FORCE-)
- new net: R5.1, U7.4 (BIAS), U7.5 (REFIN+)
- new net: R5.2, U7.6 (REFIN-), U7.7 (ISENSOR)
- new net: J8.4 (Pin_4), JP21.1 (A), U7.8 (FORCE+)
- new net: JP21.2 (C), U7.9 (FORCE2)
- new net: C18.1, J7.3 (Pin_3), U6.10 (RTDIN+)
- new net: C18.2, J7.2 (Pin_2), JP17.1 (A), U6.11 (RTDIN-)
- new net: J7.1 (Pin_1), JP17.2 (B), U6.12 (FORCE-)
- new net: R4.1, U6.4 (BIAS), U6.5 (REFIN+)
- new net: R4.2, U6.6 (REFIN-), U6.7 (ISENSOR)
- new net: J7.4 (Pin_4), JP19.1 (A), U6.8 (FORCE+)
- new net: JP19.2 (C), U6.9 (FORCE2)
- new net RTD_3_CS: U5.16 (~CS)
- new net RTD_4_CS: U6.16 (~CS)
- new net RTD_5_CS: U3.16 (~CS)
- new net RTD_6_CS: U8.16 (~CS)
- no-connect marks 2 -> 6
Other:
- moved on the sheet: C1, C2, C7, R1, U2
