File: sensorboard_due_v2/sensorboard_due.kicad_pcb (KiCad board)
At the start: 2 copper layers, 101.6 x 53.3 mm, 19 parts, among them J2 I2C_SLAVE, J3 Conn_01x03_Male, J4 GPS_UBLOX_NEO6M, J5 Micro_SD_Card, J6 Conn_01x03_Male, U1 HSCDANN001BA2A3, U2 MAX31865AAP+, U3 MAX31865AAP+

Commit message: PCB layout
Parts:
- added JP1: SolderJumper_2_Open, Jumper:SolderJumper-2_P1.3mm_Open_TrianglePad1.0x1.5mm, F.Cu at (99.1, 74.9)
- added JP2: SolderJumper_2_Open, Jumper:SolderJumper-2_P1.3mm_Open_TrianglePad1.0x1.5mm, F.Cu at (96.5, 74.9)
- added JP3: SolderJumper_2_Open, Jumper:SolderJumper-2_P1.3mm_Open_TrianglePad1.0x1.5mm, F.Cu at (94.0, 74.9)
- added JP4: SolderJumper_2_Open, Jumper:SolderJumper-2_P1.3mm_Open_TrianglePad1.0x1.5mm, F.Cu at (91.4, 74.9)
- added JP5: SolderJumper_2_Open, Jumper:SolderJumper-2_P1.3mm_Open_TrianglePad1.0x1.5mm, F.Cu at (80.0, 74.9)
- added JP6: SolderJumper_2_Open, Jumper:SolderJumper-2_P1.3mm_Open_TrianglePad1.0x1.5mm, F.Cu at (77.5, 74.9)
- added U4: MS5805-02BA01, arduino_sensors:MS5805-02BA01, F.Cu at (130.8, 83.8)
- C1, C2, C3, C4, C5, C6: footprint Capacitor_SMD:C_0402_1005Metric -> Capacitor_SMD:C_0805_2012Metric_Pad1.15x1.40mm_HandSolder
- moved C4 1.60 mm to (69.8, 76.4)
- moved C2 1.06 mm to (68.6, 90.2), turned to 180 degrees
Connections:
- H1 pad 5: (no net) -> Net-(H1-Pad5)
- H1 pad 7: (no net) -> Net-(H1-Pad7)
- H1 pad 8: (no net) -> Net-(H1-Pad8)
- H2 pad 5: (no net) -> Net-(H2-Pad5)
- H2 pad 6: (no net) -> Net-(H2-Pad6)
- H2 pad 7: (no net) -> Net-(H2-Pad7)
- H2 pad 8: (no net) -> Net-(H2-Pad8)
- J5 pad 1: (no net) -> Net-(J5-Pad1)
- J5 pad 8: (no net) -> Net-(J5-Pad8)
- J5 pad 9: (no net) -> Net-(J5-Pad9)
- PCB1 pad +5V_: (no net) -> Net-(PCB1-Pad+5V_)
- PCB1 pad 0: (no net) -> Net-(PCB1-Pad0)
- PCB1 pad 1: (no net) -> Net-(PCB1-Pad1)
- PCB1 pad 11: RTD_1_CS -> /RTD_5
- PCB1 pad 12: RTD_2_CS -> /RTD_6
- PCB1 pad 13: (no net) -> Net-(PCB1-Pad13)
- PCB1 pad 14: (no net) -> Net-(PCB1-Pad14)
- PCB1 pad 15: (no net) -> Net-(PCB1-Pad15)
- PCB1 pad 16: (no net) -> Net-(PCB1-Pad16)
- PCB1 pad 17: (no net) -> Net-(PCB1-Pad17)
- PCB1 pad 2: (no net) -> Net-(PCB1-Pad2)
- PCB1 pad 22: (no net) -> Net-(PCB1-Pad22)
- PCB1 pad 23: (no net) -> Net-(PCB1-Pad23)
- PCB1 pad 24: (no net) -> /MPU_2
- PCB1 pad 25: (no net) -> Net-(PCB1-Pad25)
- PCB1 pad 26: (no net) -> /MPU_3
- PCB1 pad 27: (no net) -> Net-(PCB1-Pad27)
- PCB1 pad 28: (no net) -> /MPU_4
- PCB1 pad 29: (no net) -> Net-(PCB1-Pad29)
- PCB1 pad 3: (no net) -> Net-(PCB1-Pad3)
- PCB1 pad 30: (no net) -> /MPU_5
- PCB1 pad 31: (no net) -> Net-(PCB1-Pad31)
- PCB1 pad 32: (no net) -> /MPU_6
- PCB1 pad 33: (no net) -> Net-(PCB1-Pad33)
- PCB1 pad 34: (no net) -> Net-(PCB1-Pad34)
- PCB1 pad 35: (no net) -> Net-(PCB1-Pad35)
- PCB1 pad 36: (no net) -> Net-(PCB1-Pad36)
- PCB1 pad 37: (no net) -> Net-(PCB1-Pad37)
- PCB1 pad 38: (no net) -> Net-(PCB1-Pad38)
- PCB1 pad 39: (no net) -> Net-(PCB1-Pad39)
- PCB1 pad 4: (no net) -> /RTD_1
- PCB1 pad 40: (no net) -> Net-(PCB1-Pad40)
- PCB1 pad 41: (no net) -> Net-(PCB1-Pad41)
- PCB1 pad 42: (no net) -> Net-(PCB1-Pad42)
- PCB1 pad 43: (no net) -> Net-(PCB1-Pad43)
- PCB1 pad 44: (no net) -> Net-(PCB1-Pad44)
- PCB1 pad 45: (no net) -> Net-(PCB1-Pad45)
- PCB1 pad 46: (no net) -> Net-(PCB1-Pad46)
- PCB1 pad 47: (no net) -> Net-(PCB1-Pad47)
- PCB1 pad 48: (no net) -> Net-(PCB1-Pad48)
- PCB1 pad 49: (no net) -> Net-(PCB1-Pad49)
- PCB1 pad 5: (no net) -> /RTD_2
- PCB1 pad 50: (no net) -> Net-(PCB1-Pad50)
- PCB1 pad 51: (no net) -> Net-(PCB1-Pad51)
- PCB1 pad 52: (no net) -> Net-(PCB1-Pad52)
- PCB1 pad 53: (no net) -> Net-(PCB1-Pad53)
- PCB1 pad 5V: (no net) -> Net-(PCB1-Pad5V)
- PCB1 pad 5V.: (no net) -> Net-(PCB1-Pad5V.)
- PCB1 pad 5V..: (no net) -> Net-(PCB1-Pad5V..)
- PCB1 pad 6: (no net) -> /RTD_3
- PCB1 pad 7: (no net) -> /RTD_4
- PCB1 pad 8: (no net) -> Net-(PCB1-Pad8)
- PCB1 pad 9: (no net) -> Net-(PCB1-Pad9)
- PCB1 pad A1: (no net) -> Net-(PCB1-PadA1)
- PCB1 pad A10: (no net) -> Net-(PCB1-PadA10)
- PCB1 pad A11: (no net) -> Net-(PCB1-PadA11)
- PCB1 pad A12: (no net) -> Net-(PCB1-PadA12)
- PCB1 pad A13: (no net) -> Net-(PCB1-PadA13)
- PCB1 pad A14: (no net) -> Net-(PCB1-PadA14)
- PCB1 pad A15: (no net) -> Net-(PCB1-PadA15)
- PCB1 pad A2: (no net) -> Net-(PCB1-PadA2)
- PCB1 pad A3: (no net) -> Net-(PCB1-PadA3)
- PCB1 pad A4: (no net) -> Net-(PCB1-PadA4)
- PCB1 pad A5: (no net) -> Net-(PCB1-PadA5)
- PCB1 pad A6: (no net) -> Net-(PCB1-PadA6)
- PCB1 pad A7: (no net) -> Net-(PCB1-PadA7)
- PCB1 pad A8: (no net) -> Net-(PCB1-PadA8)
- PCB1 pad A9: (no net) -> Net-(PCB1-PadA9)
- PCB1 pad AREF: (no net) -> Net-(PCB1-PadAREF)
- PCB1 pad GND...: (no net) -> Net-(PCB1-PadGND...)
- PCB1 pad GND....: (no net) -> Net-(PCB1-PadGND....)
- PCB1 pad GND__: (no net) -> Net-(PCB1-PadGND__)
- PCB1 pad I/OREF: (no net) -> Net-(PCB1-PadI/OREF)
- PCB1 pad N/C: (no net) -> Net-(PCB1-PadN/C)
- PCB1 pad RESET: (no net) -> Net-(PCB1-PadRESET)
- PCB1 pad RESET.: (no net) -> Net-(PCB1-PadRESET.)
- PCB1 pad VIN: (no net) -> Net-(PCB1-PadVIN)
- U1 pad 5: (no net) -> Net-(U1-Pad5)
- U1 pad 6: (no net) -> Net-(U1-Pad6)
- U1 pad 7: (no net) -> Net-(U1-Pad7)
- U1 pad 8: (no net) -> Net-(U1-Pad8)
- U2 pad 1: (no net) -> Net-(U2-Pad1)
- U2 pad 20: (no net) -> Net-(U2-Pad20)
- U3 pad 1: (no net) -> Net-(U3-Pad1)
- U3 pad 20: (no net) -> Net-(U3-Pad20)
Routing:
- net RTD_2_CS: track 15.6 -> 40.4 mm, vias 0 -> 2
- net RTD_1_CS: track 29.9 -> 46.5 mm, vias 2 -> 6
- net /SCL_MASTER: track 30.7 -> 35.6 mm
- net +3V3: track 203.1 -> 207.9 mm
- net /RTD_6: track 0.00 -> 4.46 mm
- net /RTD_5: track 0.00 -> 4.46 mm
- net /RTD_4: track 0.00 -> 4.36 mm
- net /RTD_3: track 0.00 -> 4.36 mm
- net /RTD_2: track 0.00 -> 4.36 mm
- net /RTD_1: track 0.00 -> 4.36 mm
- net /SDA_MASTER: track 33.0 -> 35.8 mm
- net GND: track 27.6 -> 28.9 mm, vias 9 -> 10
Other:
- board text added: "GPS module"
- board text added: "Populate U1 or U4 not both"
- board text added: "Use only SanDisk microSD card"

Commit message: stuff
Parts:
- added C7: 0.1u, Capacitor_SMD:C_0805_2012Metric_Pad1.15x1.40mm_HandSolder, B.Cu at (57.0, 97.0)
- added C8: 0.1u, Capacitor_SMD:C_0805_2012Metric_Pad1.15x1.40mm_HandSolder, B.Cu at (57.0, 86.0)
- added JP10: SolderJumper_2_Open, Jumper:SolderJumper-2_P1.3mm_Open_TrianglePad1.0x1.5mm, F.Cu at (64.3, 73.2)
- added JP7: SolderJumper_2_Open, Jumper:SolderJumper-2_P1.3mm_Open_TrianglePad1.0x1.5mm, B.Cu at (62.0, 76.4)
- added JP8: SolderJumper_2_Open, Jumper:SolderJumper-2_P1.3mm_Open_TrianglePad1.0x1.5mm, F.Cu at (67.1, 73.2)
- added JP9: SolderJumper_2_Open, Jumper:SolderJumper-2_P1.3mm_Open_TrianglePad1.0x1.5mm, B.Cu at (62.0, 73.7)
Connections:
- net /MPU_2 renamed Net-(PCB1-Pad24)
- net /MPU_3 renamed Net-(PCB1-Pad26)
- net /MPU_4 renamed Net-(PCB1-Pad28)
- net /MPU_5 renamed Net-(PCB1-Pad30)
- net /MPU_6 renamed Net-(PCB1-Pad32)
- net Net-(PCB1-Pad3) renamed /MIC
- J5 pad 9: Net-(J5-Pad9) -> GND
- PCB1 pad SCL1: Net-(J2-Pad2) -> /SCL_SLAVE
- PCB1 pad SDA1: Net-(J2-Pad1) -> /SDA_SLAVE
- U4 pad 2: /SDA_MASTER -> /SCL_MASTER
- U4 pad 3: /SCL_MASTER -> /SDA_MASTER
Routing:
- net /SDA_MASTER: track 35.8 -> 114.5 mm
- net /SCL_MASTER: track 35.6 -> 103.6 mm
- net /SCL_SLAVE: track 0.00 -> 2.71 mm
- net /SDA_SLAVE: track 0.00 -> 2.62 mm
- net Net-(C7-Pad2): track 20.2 -> 22.3 mm
- net Net-(C8-Pad1): track 9.18 -> 11.3 mm
- net Net-(C8-Pad2): track 18.4 -> 20.6 mm
- net Net-(C7-Pad1): track 10.1 -> 12.2 mm
- net GND: track 28.9 -> 27.9 mm, vias 10 -> 11
- net Net-(J2-Pad1): track 10.6 -> 11.3 mm
- net Net-(J2-Pad2): track 7.04 -> 7.59 mm

Commit message: incomplete pcb layout
Parts:
- removed JP1, JP2, JP3, JP4, JP5, JP6: SolderJumper_2_Open, Jumper:SolderJumper-2_P1.3mm_Open_TrianglePad1.0x1.5mm
- added C10: 0.1u, Capacitor_SMD:C_0805_2012Metric_Pad1.15x1.40mm_HandSolder, F.Cu at (117.3, 43.6)
- added C11: 0.1u, Capacitor_SMD:C_0805_2012Metric_Pad1.15x1.40mm_HandSolder, F.Cu at (98.7, 58.1)
- added C12: 0.1u, Capacitor_SMD:C_0805_2012Metric_Pad1.15x1.40mm_HandSolder, B.Cu at (84.7, 90.5)
- added C13: 0.1u, Capacitor_SMD:C_0805_2012Metric_Pad1.15x1.40mm_HandSolder, B.Cu at (104.4, 75.4)
- added C14: 0.1u, Capacitor_SMD:C_0805_2012Metric_Pad1.15x1.40mm_HandSolder, F.Cu at (90.1, 56.2)
- added C15: 0.1u, Capacitor_SMD:C_0805_2012Metric_Pad1.15x1.40mm_HandSolder, B.Cu at (86.7, 90.4)
- added C16: 0.1u, Capacitor_SMD:C_0805_2012Metric_Pad1.15x1.40mm_HandSolder, B.Cu at (104.4, 77.5)
- added C17: 0.1u, Capacitor_SMD:C_0805_2012Metric_Pad1.15x1.40mm_HandSolder, F.Cu at (112.5, 43.6)
- added C18: 0.1u, Capacitor_SMD:C_0805_2012Metric_Pad1.15x1.40mm_HandSolder, F.Cu at (108.5, 49.4)
- added C19: 0.1u, Capacitor_SMD:C_0805_2012Metric_Pad1.15x1.40mm_HandSolder, F.Cu at (123.0, 34.8)
- added C20: 0.1u, Capacitor_SMD:C_0805_2012Metric_Pad1.15x1.40mm_HandSolder, F.Cu at (117.3, 40.6)
- added C9: 0.1u, Capacitor_SMD:C_0805_2012Metric_Pad1.15x1.40mm_HandSolder, B.Cu at (87.2, 79.1)
- added J1: Conn_01x04_Male, Connector_JST:JST_XH_B4B-XH-A_1x04_P2.50mm_Vertical, F.Cu at (93.2, 93.2)
- added J7: Conn_01x04_Male, Connector_JST:JST_XH_B4B-XH-A_1x04_P2.50mm_Vertical, F.Cu at (67.3, 90.3)
- added J8: Conn_01x04_Male, Connector_JST:JST_XH_B4B-XH-A_1x04_P2.50mm_Vertical, F.Cu at (102.9, 93.2)
- added J9: Conn_01x04_Male, Connector_JST:JST_XH_B4B-XH-A_1x04_P2.50mm_Vertical, F.Cu at (67.4, 110.1)
- added JP11: SolderJumper_2_Open, Jumper:SolderJumper-2_P1.3mm_Open_Pad1.0x1.5mm, F.Cu at (62.9, 98.7)
- added JP12: SolderJumper_3_Open, Jumper:SolderJumper-3_P1.3mm_Open_Pad1.0x1.5mm, B.Cu at (61.0, 100.6)
- added JP13: SolderJumper_2_Open, Jumper:SolderJumper-2_P1.3mm_Open_Pad1.0x1.5mm, F.Cu at (117.8, 46.8)
- added JP14: SolderJumper_2_Open, Jumper:SolderJumper-2_P1.3mm_Open_Pad1.0x1.5mm, F.Cu at (122.2, 46.1)
- added JP15: SolderJumper_3_Open, Jumper:SolderJumper-3_P1.3mm_Open_Pad1.0x1.5mm, F.Cu at (73.6, 59.4)
- added JP16: SolderJumper_3_Open, Jumper:SolderJumper-3_P1.3mm_Open_Pad1.0x1.5mm, F.Cu at (73.6, 55.6)
- added JP17: SolderJumper_2_Open, Jumper:SolderJumper-2_P1.3mm_Open_Pad1.0x1.5mm, F.Cu at (112.7, 55.6)
- added JP18: SolderJumper_2_Open, Jumper:SolderJumper-2_P1.3mm_Open_Pad1.0x1.5mm, F.Cu at (107.6, 59.1)
- added JP19: SolderJumper_3_Open, Jumper:SolderJumper-3_P1.3mm_Open_Pad1.0x1.5mm, F.Cu at (79.3, 55.6)
- added JP20: SolderJumper_2_Open, Jumper:SolderJumper-2_P1.3mm_Open_Pad1.0x1.5mm, F.Cu at (108.3, 55.6)
- added JP21: SolderJumper_3_Open, Jumper:SolderJumper-3_P1.3mm_Open_Pad1.0x1.5mm, F.Cu at (79.3, 59.4)
- added JP22: SolderJumper_3_Open, Jumper:SolderJumper-3_P1.3mm_Open_Pad1.0x1.5mm, F.Cu at (84.9, 56.5)
- added R3: 400, Resistor_SMD:R_0603_1608Metric_Pad1.05x0.95mm_HandSolder, B.Cu at (84.5, 74.7)
- added R4: 400, Resistor_SMD:R_0603_1608Metric_Pad1.05x0.95mm_HandSolder, B.Cu at (84.7, 85.8)
- added R5: 400, Resistor_SMD:R_0603_1608Metric_Pad1.05x0.95mm_HandSolder, B.Cu at (99.3, 77.0)
- added R6: 400, Resistor_SMD:R_0603_1608Metric_Pad1.05x0.95mm_HandSolder, B.Cu at (84.4, 103.1)
- added U5: MAX31865AAP+, Package_SO:SSOP-20_5.3x7.2mm_P0.65mm, F.Cu at (83.6, 80.6)
- added U6: MAX31865AAP+, Package_SO:SSOP-20_5.3x7.2mm_P0.65mm, F.Cu at (83.6, 91.0)
- added U7: MAX31865AAP+, Package_SO:SSOP-20_5.3x7.2mm_P0.65mm, F.Cu at (104.8, 78.5)
- added U8: MAX31865AAP+, Package_SO:SSOP-20_5.3x7.2mm_P0.65mm, F.Cu at (83.6, 110.8)
- C1, C2, C4, R2: moved to B.Cu
- C8: moved to F.Cu
- J3, J6: value Conn_01x03_Male -> Conn_01x04_Male; footprint Connector_Molex_70553:70553-0002_3P -> Connector_JST:JST_XH_B4B-XH-A_1x04_P2.50mm_Vertical
- moved C8 61.6 mm to (108.5, 52.3), turned to 0 degrees
- moved JP10 37.5 mm to (32.8, 52.9)
- moved JP8 37.5 mm to (35.6, 52.9)
- moved C3 36.0 mm to (94.0, 59.2), turned to 0 degrees
- moved C1 33.3 mm to (93.2, 75.7), turned to 0 degrees
- moved R1 33.1 mm to (90.4, 73.7), turned to 0 degrees
- moved C5 28.6 mm to (32.5, 102.9)
- moved U2 28.1 mm to (93.5, 78.5)
- moved C2 27.6 mm to (93.2, 77.7), turned to 0 degrees
- moved J5 22.1 mm to (54.9, 87.6)
- moved U3 21.7 mm to (83.6, 100.9), turned to 270 degrees
- moved H1 16.7 mm to (113.8, 100.1)
- moved R2 15.0 mm to (84.5, 95.2)
- moved C4 13.9 mm to (83.5, 79.2), turned to 180 degrees
- moved J6 10.8 mm to (67.3, 80.4), turned to 0 degrees
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Connections:
- C8 pad 1: Net-(C8-Pad1) -> +3V3
- C8 pad 2: Net-(C8-Pad2) -> GND
- J3 pad 1: Net-(C7-Pad2) -> Net-(J3-Pad1)
- J3 pad 2: Net-(C7-Pad1) -> Net-(C10-Pad2)
- J3 pad 3: Net-(J3-Pad3) -> Net-(C10-Pad1)
- J6 pad 1: Net-(C8-Pad2) -> Net-(J6-Pad1)
- J6 pad 2: Net-(C8-Pad1) -> Net-(C11-Pad2)
- J6 pad 3: Net-(J6-Pad3) -> Net-(C11-Pad1)
- PCB1 pad 11: /RTD_5 -> Net-(PCB1-Pad11)
- PCB1 pad 12: /RTD_6 -> Net-(PCB1-Pad12)
- PCB1 pad 2: Net-(PCB1-Pad2) -> RTD_1_CS
- PCB1 pad 3: /MIC -> RTD_2_CS
- PCB1 pad 4: /RTD_1 -> Net-(PCB1-Pad4)
- PCB1 pad 5: /RTD_2 -> Net-(PCB1-Pad5)
- PCB1 pad 6: /RTD_3 -> Net-(PCB1-Pad6)
- PCB1 pad 7: /RTD_4 -> RTD_3_CS
- PCB1 pad A1: Net-(PCB1-PadA1) -> RTD_6_CS
- PCB1 pad A2: Net-(PCB1-PadA2) -> RTD_5_CS
- PCB1 pad A3: Net-(PCB1-PadA3) -> RTD_4_CS
- U2 pad 12: Net-(C7-Pad2) -> Net-(J1-Pad1)
- U2 pad 16: RTD_1_CS -> RTD_2_CS
- U2 pad 8: Net-(J3-Pad3) -> Net-(J1-Pad4)
- U2 pad 9: Net-(J3-Pad3) -> Net-(JP12-Pad2)
- U3 pad 10: Net-(C8-Pad1) -> Net-(C10-Pad1)
- U3 pad 11: Net-(C8-Pad2) -> Net-(C10-Pad2)
- U3 pad 12: Net-(C8-Pad2) -> Net-(J3-Pad1)
- U3 pad 16: RTD_2_CS -> RTD_5_CS
- U3 pad 8: Net-(J6-Pad3) -> Net-(J3-Pad4)
- U3 pad 9: Net-(J6-Pad3) -> Net-(JP15-Pad2)
Routing:
- net +3V3: track 207.9 -> 12.6 mm, vias 4 -> 6
- net /SDA_MASTER: track 114.5 -> 0.00 mm
- net /SCL_MASTER: track 103.6 -> 0.00 mm
- net /SD_CS: track 48.1 -> 0.00 mm
- net MISO: track 81.0 -> 120.8 mm, vias 2 -> 5
- net RTD_4_CS: track 0.00 -> 35.0 mm
- net RTD_1_CS: track 46.5 -> 11.7 mm, vias 6 -> 0
- net RTD_2_CS: track 40.4 -> 10.8 mm, vias 2 -> 0
- net /MPU_1: track 28.0 -> 0.00 mm, vias 2 -> 0
- net RTD_5_CS: track 0.00 -> 25.9 mm
- net SCK: track 80.5 -> 103.4 mm, vias 2 -> 5
- net Net-(C8-Pad2): track 20.6 -> 0.00 mm, vias 1 -> 0
- net RTD_6_CS: track 0.00 -> 18.3 mm
- net Net-(J8-Pad1): track 0.00 -> 16.3 mm
- net Net-(J1-Pad1): track 0.00 -> 15.6 mm
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- removed copper zone on B.Cu, net GND
Other:
- copper layers 2 -> 4
- board text removed: "Use only SanDisk microSD card"
